File: SSL Base SMD - v12/SSL Base SMD - v12.kicad_pcb (KiCad board)
At the start: 2 copper layers, 164.9 x 152 mm, 155 parts, among them J1 NRF24L01, Q1 2N3904, U3 STM32F401VETx, U5 LM338T

Commit message: Add files via upload
Parts:
- removed J1: NRF24L01, Connector_PinSocket_2.54mm:PinSocket_2x04_P2.54mm_Vertical
- C1: value 10u -> 100u
- Q1: footprint Package_TO_SOT_SMD:SOT-23 -> Package_TO_SOT_THT:TO-92L_Inline_Wide
- R1: footprint Resistor_SMD:R_0805_2012Metric -> Resistor_THT:R_Axial_DIN0204_L3.6mm_D1.6mm_P2.54mm_Vertical
- moved Q1 3.28 mm to (155.0, 148.8), turned to 90 degrees
- moved R1 1.94 mm to (152.1, 143.8)
Routing:
- net Net-(BZ1-+): track 14.2 -> 16.7 mm
- net Net-(Q1-B): track 2.11 -> 3.88 mm
- net H1_M3: track 60.6 -> 59.6 mm
- net Buzzer: track 87.7 -> 86.9 mm
