File: SSL Base SMD - v12/SSL Base SMD - v12.kicad_sch (KiCad schematic)
At the start: 155 parts, among them J1 NRF24L01, J21 Chute1, Q1 2N3904, U3 STM32F401VETx, U5 LM338T

Commit message: Add files via upload
Parts:
- removed J1: NRF24L01, Connector_PinSocket_2.54mm:PinSocket_2x04_P2.54mm_Vertical, symbol Connector_Generic:Conn_02x04_Counter_Clockwise
- C1: value 10u -> 100u
- Q1: footprint Package_TO_SOT_SMD:SOT-23 -> Package_TO_SOT_THT:TO-92L_Inline_Wide
- R1: footprint Resistor_SMD:R_0805_2012Metric -> Resistor_THT:R_Axial_DIN0204_L3.6mm_D1.6mm_P2.54mm_Vertical
Changed lines of the file:
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@@
     )
   )
-  (global_label "SPI1_SCK" (shape input) (at 84.074 114.046 180) (fields_autoplaced)
-    (effects (font (size 1.27 1.27)) (justify right))
-    (property "Intersheetrefs" "${INTERSHEET_REFS}" (at 72.1573 114.046 0)
-      (effects (font (size 1.27 1.27)) (justify right) hide)
-    )
-  )
   (global_label "DISPARO NORMAL" (shape input) (at 102.362 98.806 180) (fields_autoplaced)
     (effects (font (size 1.27 1.27)) (justify right))
@@
     )
   )
-  (global_label "SPI1_MOSI" (shape input) (at 84.074 116.586 180) (fields_autoplaced)
-    (effects (font (size 1.27 1.27)) (justify right))
-    (property "Intersheetrefs" "${INTERSHEET_REFS}" (at 71.3106 116.586 0)
-      (effects (font (size 1.27 1.27)) (justify right) hide)
-    )
-  )
   (global_label "HALL1_M2" (shape input) (at 422.91 27.432 0) (fields_autoplaced)
     (effects (font (size 1.27 1.27)) (justify left))
@@
     )
   )
-  (global_label "IO0" (shape input) (at 51.562 42.672 0) (fields_autoplaced)
-    (effects (font (size 1.27 1.27)) (justify left))
-    (property "Intersheetrefs" "${INTERSHEET_REFS}" (at 57.6126 42.672 0)
-      (effects (font (size 1.27 1.27)) (justify left) hide)
-    )
-  )
   (global_label "18V" (shape input) (at 338.328 22.352 180) (fields_autoplaced)
     (effects (font (size 1.27 1.27)) (justify right))
@@
     )
   )
-  (global_label "SPI1_MISO" (shape input) (at 86.36 55.626 180) (fields_autoplaced)
-    (effects (font (size 1.27 1.27)) (justify right))
-    (property "Intersheetrefs" "${INTERSHEET_REFS}" (at 73.5966 55.626 0)
-      (effects (font (size 1.27 1.27)) (justify right) hide)
-    )
-  )
   (global_label "5V" (shape input) (at 186.944 51.816 180) (fields_autoplaced)
     (effects (font (size 1.27 1.27)) (justify right))
@@
       (effects (font (size 1.27 1.27)))
     )
-    (property "Footprint" "Resistor_SMD:R_0805_2012Metric" (at 246.888 236.982 90)
+    (property "Footprint" "Resistor_THT:R_Axial_DIN0204_L3.6mm_D1.6mm_P2.54mm_Vertical" (at 246.888 236.982 90)
       (effects (font (size 1.27 1.27)) hide)
     )
@@
       (effects (font (size 1.27 1.27)) (justify left))
     )
-    (property "Footprint" "Package_TO_SOT_SMD:SOT-23" (at 260.858 240.665 0)
+    (property "Footprint" "Package_TO_SOT_THT:TO-92L_Inline_Wide" (at 260.858 240.665 0)
       (effects (font (size 1.27 1.27) italic) (justify left) hide)
     )
@@
     )
   )
-  (symbol (lib_id "Connector_Generic:Conn_02x04_Counter_Clockwise") (at 45.974 82.804 0) (unit 1)
-    (in_bom yes) (on_board yes) (dnp no) (fields_autoplaced)
-    (property "Reference" "J1" (at 47.244 74.93 0)
-      (effects (font (size 1.27 1.27)))
-    )
-    (property "Value" "NRF24L01" (at 47.244 77.47 0)
-      (effects (font (size 1.27 1.27)))
-    )
-    (property "Footprint" "Connector_PinSocket_2.54mm:PinSocket_2x04_P2.54mm_Vertical" (at 45.974 82.804 0)
-      (effects (font (size 1.27 1.27)) hide)
-    )
-    (property "Datasheet" "~" (at 45.974 82.804 0)
-      (effects (font (size 1.27 1.27)) hide)
-    )
-    (pin "1")
-    (pin "2")
-    (pin "3")
-    (pin "4")
-    (pin "5")
-    (pin "6")
-    (pin "7")
-    (pin "8")
-    (instances
-      (project "SSL Base SMD - v12"
-        (path "/82e4a3bf-8a14-4453-a27e-85b488823db3"
-          (reference "J1") (unit 1)
-        )
-      )
-    )
-  )
   (symbol (lib_id "Diode:1N5408") (at 17.018 181.102 270) (unit 1)
     (in_bom yes) (on_board yes) (dnp no) (fields_autoplaced)
@@
       (effects (font (size 1.27 1.27)) (justify right))
     )
-    (property "Value" "10u" (at 90.17 163.576 0)
+    (property "Value" "100u" (at 90.17 163.576 0)
       (effects (font (size 1.27 1.27)) (justify right))
     )
