File: Placa do Chute v5 - PTH/Placa do Chute v5 - PTH.kicad_pcb (KiCad board)
At the start: 2 copper layers, 84.9 x 40 mm, 31 parts, among them J1 Conn_02x11x2_Pin_Maraca, Q1 IRFP260N, Q2 IRFP260N, Q3 IRFP260N, U1 OPTO PWM, U2 OPTO DISPARO KICK, U3 OPTO DISPARO

Commit message: Add files via upload
Parts:
- Descarregar2: moved to B.Cu
- moved Descarregar2 4.51 mm to (192.4, 113.8), turned to 180 degrees
- moved R7 1.50 mm to (177.3, 90.9)
- moved R12 0.66 mm to (174.2, 80.7)
- moved R10 0.36 mm to (149.0, 95.2)
- renumbered U1 to Carga1, U2 to Chip_Kick1, U3 to Chute1, Q1 to QCarga1, Q3 to QChip_Kick3, Q2 to QChute2
Connections:
- Descarregar2 pad 1: 18V -> Net-(Descarregar2-Pad1)
- Descarregar2 pad 2: Net-(Descarregar2-Pad2) -> 18V
- R9 pad 1: Net-(Descarregar2-Pad2) -> Net-(Descarregar2-Pad1)
Routing:
- net Net-(Descarregar2-Pad1): track 0.00 -> 20.7 mm, vias 0 -> 1
- net Net-(Descarregar2-Pad2): track 20.7 -> 0.00 mm, vias 1 -> 0
- net Net-(D7-A): track 40.6 -> 59.6 mm
- net Net-(Chip_Kick1-Pad1): track 46.4 -> 47.0 mm
- net DISPARO CHIP KICK: track 50.6 -> 51.1 mm
- net SOLENOIDE1_2: track 122.6 -> 123.1 mm
- net Net-(D8-A): track 31.1 -> 30.6 mm

Commit message: Add files via upload
Parts:
- Descarregar1: renamed from Descarregar2; value 1825910-6 -> FSMRA4JH04
