File: Placa do Chute v5 - PTH/Placa do Chute v5 - PTH.kicad_sch (KiCad schematic)
At the start: 31 parts, among them J1 Conn_02x11x2_Pin_Maraca, Q1 IRFP260N, Q2 IRFP260N, Q3 IRFP260N, U1 OPTO PWM, U2 OPTO DISPARO KICK, U3 OPTO DISPARO

Commit message: Add files via upload
Parts:
- renumbered U1 to Carga1, U2 to Chip_Kick1, U3 to Chute1, Q1 to QCarga1, Q3 to QChip_Kick3, Q2 to QChute2
Connections:
- net 18V: now also Descarregar2.2; no longer Descarregar2.1
- net at R9.1: now also Descarregar2.1; no longer Descarregar2.2
Changed lines of the file:
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@@
-    (stroke (width 0) (type default))
-  )
-  (wire (pts (xy 168.402 92.964) (xy 170.18 92.964))
     (stroke (width 0) (type default))
   )
@@
     (stroke (width 0) (type default))
   )
+  (wire (pts (xy 170.18 90.17) (xy 168.402 90.17))
+    (stroke (width 0) (type default))
+  )
   (wire (pts (xy 136.398 52.324) (xy 136.398 49.784))
     (stroke (width 0) (type default))
@@
     (stroke (width 0) (type default))
   )
-  (wire (pts (xy 170.18 92.964) (xy 170.18 95.25))
-    (stroke (width 0) (type default))
-  )
   (wire (pts (xy 140.716 52.324) (xy 136.398 52.324))
     (stroke (width 0) (type default))
@@
     (stroke (width 0) (type default))
   )
-  (wire (pts (xy 168.402 95.25) (xy 168.402 92.964))
+  (wire (pts (xy 168.402 90.17) (xy 168.402 95.25))
     (stroke (width 0) (type default))
   )
@@
     )
   )
+  (global_label "18V" (shape input) (at 170.18 95.25 180) (fields_autoplaced)
+    (effects (font (size 1.27 1.27)) (justify right))
+    (property "Intersheetrefs" "${INTERSHEET_REFS}" (at 163.7666 95.25 0)
+      (effects (font (size 1.27 1.27)) (justify right) hide)
+    )
+  )
   (global_label "SOLENOIDE2_2" (shape input) (at 126.238 45.466 180) (fields_autoplaced)
     (effects (font (size 1.27 1.27)) (justify right))
@@
     (property "Intersheetrefs" "${INTERSHEET_REFS}" (at 40.9635 49.53 0)
       (effects (font (size 1.27 1.27)) (justify right) hide)
-    )
-  )
-  (global_label "18V" (shape input) (at 170.18 90.17 90) (fields_autoplaced)
-    (effects (font (size 1.27 1.27)) (justify left))
-    (property "Intersheetrefs" "${INTERSHEET_REFS}" (at 170.18 83.7566 90)
-      (effects (font (size 1.27 1.27)) (justify left) hide)
     )
   )
@@
   (symbol (lib_id "IRFP260N:IRFP260N") (at 128.778 52.324 0) (mirror y) (unit 1)
     (in_bom yes) (on_board yes) (dnp no)
-    (property "Reference" "Q3" (at 123.444 51.689 0)
+    (property "Reference" "QChip_Kick3" (at 123.444 51.689 0)
       (effects (font (size 1.27 1.27)) (justify left))
     )
@@
       (project "Placa do Chute v5 - PTH"
         (path "/1de9637d-97cd-4863-af99-42f1b5fd7dcb"
-          (reference "Q3") (unit 1)
+          (reference "QChip_Kick3") (unit 1)
         )
       )
@@
   (symbol (lib_id "IRFP260N:IRFP260N") (at 70.358 85.344 0) (unit 1)
     (in_bom yes) (on_board yes) (dnp no) (fields_autoplaced)
-    (property "Reference" "Q1" (at 75.692 84.709 0)
-      (effects (font (size 1.27 1.27)) (justify left))
-    )
-    (property "Value" "IRFP260N" (at 75.692 87.249 0)
+    (property "Reference" "QCarga1" (at 76.2 84.709 0)
+      (effects (font (size 1.27 1.27)) (justify left))
+    )
+    (property "Value" "IRFP260N" (at 76.2 87.249 0)
       (effects (font (size 1.27 1.27)) (justify left))
     )
@@
       (project "Placa do Chute v5 - PTH"
         (path "/1de9637d-97cd-4863-af99-42f1b5fd7dcb"
-          (reference "Q1") (unit 1)
+          (reference "QCarga1") (unit 1)
         )
       )
@@
   (symbol (lib_id "Isolator:4N25") (at 149.606 96.52 0) (mirror y) (unit 1)
     (in_bom yes) (on_board yes) (dnp no)
-    (property "Reference" "U3" (at 149.606 88.646 0)
+    (property "Reference" "Chute1" (at 149.606 88.646 0)
       (effects (font (size 1.27 1.27)))
     )
@@
       (project "Placa do Chute v5 - PTH"
         (path "/1de9637d-97cd-4863-af99-42f1b5fd7dcb"
-          (reference "U3") (unit 1)
+          (reference "Chute1") (unit 1)
         )
       )
@@
   (symbol (lib_id "Isolator:4N25") (at 51.816 87.884 0) (unit 1)
     (in_bom yes) (on_board yes) (dnp no) (fields_autoplaced)
-    (property "Reference" "U1" (at 51.816 80.772 0)
-      (effects (font (size 1.27 1.27)))
-    )
-    (property "Value" "OPTO PWM" (at 51.816 83.312 0)
+    (property "Reference" "Carga1" (at 51.816 80.01 0)
+      (effects (font (size 1.27 1.27)))
+    )
+    (property "Value" "OPTO PWM" (at 51.816 82.55 0)
       (effects (font (size 1.27 1.27)))
     )
@@
       (project "Placa do Chute v5 - PTH"
         (path "/1de9637d-97cd-4863-af99-42f1b5fd7dcb"
-          (reference "U1") (unit 1)
+          (reference "Carga1") (unit 1)
         )
       )
@@
   (symbol (lib_id "Isolator:4N25") (at 148.336 52.324 0) (mirror y) (unit 1)
     (in_bom yes) (on_board yes) (dnp no)
-    (property "Reference" "U2" (at 148.336 44.196 0)
+    (property "Reference" "Chip_Kick1" (at 148.336 44.196 0)
       (effects (font (size 1.27 1.27)))
     )
@@
       (project "Placa do Chute v5 - PTH"
         (path "/1de9637d-97cd-4863-af99-42f1b5fd7dcb"
-          (reference "U2") (unit 1)
+          (reference "Chip_Kick1") (unit 1)
         )
       )
@@
   (symbol (lib_id "IRFP260N:IRFP260N") (at 128.524 96.52 0) (mirror y) (unit 1)
     (in_bom yes) (on_board yes) (dnp no)
-    (property "Reference" "Q2" (at 123.19 95.885 0)
+    (property "Reference" "QChute2" (at 123.19 95.885 0)
       (effects (font (size 1.27 1.27)) (justify left))
     )
@@
       (project "Placa do Chute v5 - PTH"
         (path "/1de9637d-97cd-4863-af99-42f1b5fd7dcb"
-          (reference "Q2") (unit 1)
-        )
-      )
+          (reference "QChute2") (unit 1)
+        )
+      )

Commit message: Add files via upload
Parts:
- removed Descarregar2: 1825910-6, Maraca:FSMRA4JH04, symbol Maraca:1825910-6
- added Descarregar1: FSMRA4JH04, Maraca:FSMRA4JH04, symbol FSMRA4JH04:FSMRA4JH04
Connections:
- net 18V: now also Descarregar1.2 (NO)
- net GND: now also Descarregar1.3 (MH1), Descarregar1.4 (MH2)
- net at R9.1: now also Descarregar1.1 (COM)
Other:
- moved on the sheet: D5, R9
