File: Placa do Chute v6 - PTH/Placa do Chute v6 - PTH.kicad_pcb (KiCad board)
At the start: 2 copper layers, 84.9 x 40 mm, 33 parts, among them J1 Conn_02x11x2_Pin_Maraca

Commit message: Add files via upload
Routing:
- net Net-(Chip_Kick1-Pad4): track 34.3 -> 37.3 mm
- net DISPARO NORMAL: track 30.2 -> 31.2 mm
- net ADC_Chute: track 39.8 -> 39.1 mm
- net Net-(D5-A): track 9.60 -> 9.03 mm
- net GND: vias 36 -> 28

Commit message: Add files via upload
Parts:
- renumbered QCarga1 to CargaQ1, QChip_Kick3 to Chip_KickQ3, QChute2 to ChuteQ2
Changed lines of the file:
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@@
     (property "Sheetname" "")
     (attr through_hole)
-    (fp_text reference "QCarga1" (at 2.770152 3.3075) (layer "F.SilkS")
+    (fp_text reference "CargaQ1" (at 2.770152 3.3075) (layer "F.SilkS")
         (effects (font (size 1 1) (thickness 0.15)))
     )
@@
     (property "Sheetname" "")
     (attr through_hole)
-    (fp_text reference "QChip_Kick3" (at -2.559848 3.0475) (layer "F.SilkS")
+    (fp_text reference "Chip_KickQ3" (at -4.429848 3.4375) (layer "F.SilkS")
         (effects (font (size 1 1) (thickness 0.15)))
     )
@@
     (property "Sheetname" "")
     (attr through_hole)
-    (fp_text reference "QChute2" (at -0.039848 3.62) (layer "B.SilkS")
+    (fp_text reference "ChuteQ2" (at -0.039848 3.62) (layer "B.SilkS")
         (effects (font (size 1 1) (thickness 0.15)) (justify mirror))
     )
