File: Placa do Chute v6 - PTH/Placa do Chute v6 - PTH.kicad_sch (KiCad schematic)
At the start: 33 parts, among them J1 Conn_02x11x2_Pin_Maraca

Commit message: Add files via upload
Parts:
- renumbered QCarga1 to CargaQ1, QChip_Kick3 to Chip_KickQ3, QChute2 to ChuteQ2
Changed lines of the file:
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@@
   (symbol (lib_id "IRFP260N:IRFP260N") (at 128.778 52.324 0) (mirror y) (unit 1)
     (in_bom yes) (on_board yes) (dnp no)
-    (property "Reference" "QChip_Kick3" (at 123.444 51.689 0)
+    (property "Reference" "Chip_KickQ3" (at 123.444 51.689 0)
       (effects (font (size 1.27 1.27)) (justify left))
     )
@@
       (project "Placa do Chute v6 - PTH"
         (path "/1de9637d-97cd-4863-af99-42f1b5fd7dcb"
-          (reference "QChip_Kick3") (unit 1)
+          (reference "Chip_KickQ3") (unit 1)
         )
       )
@@
   (symbol (lib_id "IRFP260N:IRFP260N") (at 70.358 85.344 0) (unit 1)
     (in_bom yes) (on_board yes) (dnp no) (fields_autoplaced)
-    (property "Reference" "QCarga1" (at 76.2 84.709 0)
+    (property "Reference" "CargaQ1" (at 76.2 84.709 0)
       (effects (font (size 1.27 1.27)) (justify left))
     )
@@
       (project "Placa do Chute v6 - PTH"
         (path "/1de9637d-97cd-4863-af99-42f1b5fd7dcb"
-          (reference "QCarga1") (unit 1)
+          (reference "CargaQ1") (unit 1)
         )
       )
@@
   (symbol (lib_id "IRFP260N:IRFP260N") (at 128.524 96.52 0) (mirror y) (unit 1)
     (in_bom yes) (on_board yes) (dnp no)
-    (property "Reference" "QChute2" (at 123.19 95.885 0)
+    (property "Reference" "ChuteQ2" (at 123.19 95.885 0)
       (effects (font (size 1.27 1.27)) (justify left))
     )
@@
       (project "Placa do Chute v6 - PTH"
         (path "/1de9637d-97cd-4863-af99-42f1b5fd7dcb"
-          (reference "QChute2") (unit 1)
-        )
-      )
+          (reference "ChuteQ2") (unit 1)
+        )
+      )
